Commit message: prefixed urdf packages with "xpp_"

File: robots/hyq/xpp_hyq_biped_description/urdf/biped.urdf (robot description, URDF)
Before this commit: robot biped, 7 links, 6 joints
Links:
- link L_hipassembly: geometry visual mesh filename=package://xpp_hyq_biped_description/meshes/leg/hip.dae scale=1 1 1
- link L_lowerleg: geometry visual mesh filename=package://xpp_hyq_biped_description/meshes/leg/lower.dae scale=1 1 1
- link L_upperleg: geometry visual mesh filename=package://xpp_hyq_biped_description/meshes/leg/upper.dae scale=1 1 1
- link R_hipassembly: geometry visual mesh filename=package://xpp_hyq_biped_description/meshes/leg/hip.dae scale=1 1 1
- link R_lowerleg: geometry visual mesh filename=package://xpp_hyq_biped_description/meshes/leg/lower.dae scale=1 1 1
- link R_upperleg: geometry visual mesh filename=package://xpp_hyq_biped_description/meshes/leg/upper.dae scale=1 1 1

File: robots/hyq/xpp_hyq_description/urdf/trunk.urdf.xacro (robot description, xacro)
@@ -21,23 +21,15 @@
 		<!-- Trunk link -->
 		<link name="trunk">
-			<inertial>
-				<origin xyz="${xcom_trunk} ${ycom_trunk} ${zcom_trunk}"/>
-				<mass value="${m_trunk}"/>
-				<inertia ixx="${ixx_trunk}" iyy="${iyy_trunk}" izz="${izz_trunk}"
-						 ixy="${ixy_trunk}" ixz="${ixz_trunk}" iyz="${iyz_trunk}"/>
-			</inertial>
 			<visual>
 				<geometry>
-					<mesh filename="package://hyqb_description/meshes/trunk/trunk.dae" scale="1 1 1"/>
+					<mesh filename="package://xpp_hyq_description/meshes/trunk/trunk.dae" scale="1 1 1"/>
 				</geometry>
 			</visual>
 			<collision>
 				<geometry>
-					<mesh filename="package://hyqb_description/meshes/trunk/trunk.dae" scale="1 1 1"/>
+					<mesh filename="package://xpp_hyq_description/meshes/trunk/trunk.dae" scale="1 1 1"/>
 				</geometry>
 			</collision>
 		</link>
-		<!-- Extensions -->
-		<xacro:trunk_gazebo name="trunk"/>
 	</xacro:macro>
 </robot>

File: robots/hyq/xpp_hyq_monoped_description/urdf/monoped.urdf (robot description, URDF)
Before this commit: robot monoped, 4 links, 3 joints
Links:
- link hipassembly: geometry visual mesh filename=package://xpp_hyq_monoped_description/meshes/leg/hip.dae scale=1 1 1
- link lowerleg: geometry visual mesh filename=package://xpp_hyq_monoped_description/meshes/leg/lower.dae scale=1 1 1
- link upperleg: geometry visual mesh filename=package://xpp_hyq_monoped_description/meshes/leg/upper.dae scale=1 1 1
